File: design/Max98357I2SAmp/Max98357I2SAmp.kicad_pcb (KiCad board)
At the start: 2 copper layers, 20.6 x 20.6 mm, 9 parts, among them J1 Conn_01x07, J2 Conn_01x02, U1 MAX98357A

Commit message: adjustement and gerber files
Parts:
- removed C4: C, Capacitor_SMD:C_0805_2012Metric
- added C2: 100nF, Capacitor_SMD:C_0603_1608Metric_Pad1.08x0.95mm_HandSolder, F.Cu at (49.9, 36.0)
- C1, C3: value C -> 100nF; footprint Capacitor_SMD:C_0805_2012Metric -> Capacitor_SMD:C_0603_1608Metric_Pad1.08x0.95mm_HandSolder
- FB1, FB2: footprint Capacitor_SMD:C_0805_2012Metric -> Capacitor_SMD:C_0603_1608Metric_Pad1.08x0.95mm_HandSolder
- J1: footprint Connector_JST:JST_SH_BM07B-SRSS-TB_1x07-1MP_P1.00mm_Vertical -> Connector_JST:JST_SH_SM07B-SRSS-TB_1x07-1MP_P1.00mm_Horizontal
- J2: footprint Connector_JST:JST_SH_BM02B-SRSS-TB_1x02-1MP_P1.00mm_Vertical -> Connector_JST:JST_PH_S2B-PH-SM4-TB_1x02-1MP_P2.00mm_Horizontal
- R1: value R -> 1MΩ; footprint Resistor_SMD:R_0805_2012Metric -> Resistor_SMD:R_0603_1608Metric_Pad0.98x0.95mm_HandSolder
- moved J2 12.1 mm to (60.0, 40.2), turned to 90 degrees
- moved C3 8.18 mm to (49.9, 44.0)
- moved C1 2.94 mm to (45.7, 39.8)
- moved R1 2.89 mm to (41.9, 44.5), turned to -90 degrees
- moved FB1 2.86 mm to (45.6, 43.9)
- moved FB2 2.86 mm to (45.7, 36.1)
- moved U1 2.86 mm to (41.1, 40.0)
- moved J1 1.18 mm to (33.7, 40.3), turned to -90 degrees
Connections:
- C3 pad 1: Net-(J2-Pin_1) -> Net-(J2-Pin_2)
- R1 pad 1: VDD -> SD_MODE
- R1 pad 2: SD_MODE -> VDD
Routing:
- net Net-(J2-Pin_1): track 5.88 -> 12.0 mm
- net Net-(J2-Pin_2): track 5.94 -> 11.8 mm
- net GND: track 5.85 -> 9.34 mm, vias 0 -> 2
- net OUTP: track 8.97 -> 12.0 mm
- net GAIN: track 5.51 -> 6.53 mm
- net SD_MODE: track 8.59 -> 9.61 mm
- net DIN: track 4.58 -> 5.60 mm
- net BCLK: track 4.27 -> 5.29 mm
- net LRCLK: track 4.46 -> 5.48 mm
- net VDD: track 15.5 -> 16.3 mm
Other:
- board size 20.6 x 20.6 mm -> 35.8 x 20.6 mm
