File: design/Max98357I2SAmp/Max98357I2SAmp.kicad_sch (KiCad schematic)
At the start: 9 parts, among them J1 Conn_01x07, J2 Conn_01x02, U1 MAX98357A

Commit message: adjustement and gerber files
Parts:
- removed C4: C, Capacitor_SMD:C_0805_2012Metric, symbol Device:C
- added C2: 100nF, Capacitor_SMD:C_0603_1608Metric_Pad1.08x0.95mm_HandSolder, symbol Device:C
- C1, C3: value C -> 100nF; footprint Capacitor_SMD:C_0805_2012Metric -> Capacitor_SMD:C_0603_1608Metric_Pad1.08x0.95mm_HandSolder
- FB1, FB2: footprint Capacitor_SMD:C_0805_2012Metric -> Capacitor_SMD:C_0603_1608Metric_Pad1.08x0.95mm_HandSolder
- J1: footprint Connector_JST:JST_SH_BM07B-SRSS-TB_1x07-1MP_P1.00mm_Vertical -> Connector_JST:JST_SH_SM07B-SRSS-TB_1x07-1MP_P1.00mm_Horizontal
- J2: footprint Connector_JST:JST_SH_BM02B-SRSS-TB_1x02-1MP_P1.00mm_Vertical -> Connector_JST:JST_PH_S2B-PH-SM4-TB_1x02-1MP_P2.00mm_Horizontal
- R1: value R -> 1MΩ; footprint Resistor_SMD:R_0805_2012Metric -> Resistor_SMD:R_0603_1608Metric_Pad0.98x0.95mm_HandSolder
Connections:
- net GND: now also C2.2
- net SD_MODE: now also R1.1; no longer R1.2
- net VDD: now also R1.2; no longer R1.1
- net at FB2.2, J2.1 (Pin_1): now also C2.1; no longer C3.1
- net at FB1.2, J2.2 (Pin_2): now also C3.1
Other:
- moved on the sheet: U1
